Commit message: Updated launch files for simulation and real world testing

File: final_ws/src/map_sim/urdf/sick_lms291.urdf.xacro (robot description, xacro)
@@ -21,4 +21,5 @@
       <origin xyz="0 0 0" rpy="0 0 ${PI/1}" />
       <geometry>
+        <!-- sphere radius="0.05" / -->
         <mesh filename="package://map_sim/meshes/lms291_asm.stl" scale="0.001 0.001 0.001" />
       </geometry>
@@ -28,5 +29,6 @@
       <origin xyz="0 0 0" rpy="0 0 0" />
       <geometry>
-        <box size="0.155 0.156 0.185"/>
+        <sphere radius="0.05" />
+        <!-- box size="0.155 0.156 0.185"/ -->
       </geometry>
     </collision>
@@ -70,6 +72,6 @@
     <material>Gazebo/Blue</material>
     <turnGravityOff>true</turnGravityOff>
-    <sensor type="gpu_ray" name="lms291_sensor">
-      <pose>0 0 0 0 0 0</pose>
+    <sensor type="ray" name="laser">
+      <pose>0 0 5 0 0 0</pose>
       <visualize>true</visualize>
       <update_rate>40</update_rate>
@@ -94,6 +96,6 @@
         </noise>
       </ray>
-      <plugin name="gazebo_ros_laser" filename="libgazebo_ros_gpu_laser.so">
-        <topicName>scan</topicName>
+      <plugin name="laser_plug" filename="libgazebo_ros_laser.so">
+        <topicName>/scan</topicName>
         <frameName>lms291</frameName>
       </plugin>
